File: EPS_Lobosat_V1.kicad_sch (KiCad schematic)
At the start: 56 parts, among them Q1 FS8205A, Q2 FS8205A, U1 LMZM33602RLRR, U10 STPS140ZY, U2 LT3652EMSE_PBF, U3 DW01A, U5 STPS140ZY, U6 ADS1015IRUGR, U7 STPS140ZY, U8 LT3652EMSE_PBF, U9 DW01A

Commit message: Snapshot: last hand-drawn schematic + Claude desktop kit, before restructure
Co-Authored-By: Claude Opus 5.5 <noreply@anthropic.com>
Parts:
- removed BT1: Battery, symbol Device:Battery
- removed BT2: SM141K06L, SM141K06L:SOLAR_SM141K06L, symbol SM141K06L:SM141K06L
- removed C1: GRM188R72A104KA35D, GRM188R72A104KA35D:CAPC1608X90N, symbol GRM188R72A104KA35D:GRM188R72A104KA35D
- removed C2: 10uF, symbol Device:C
- removed C3, C7: 0.1uF, symbol Device:C
- removed C4: C, symbol Device:C
- removed CR1: CMSH3-40MA TR13 PBFREE, CR_SMA-CMSH3-40MA_CNS, symbol CSMH:CMSH3-40MA_TR13_PBFREE
- removed D1: SMBJ15A TVS DIODE 15VWM, symbol Device:D
- removed D2: SS34, SS34:DIOM7959X265N, symbol SS34:SS34
- removed L2: 4.7µH, ≥3A, symbol Device:L
- removed Q1, Q2: FS8205A, FS8205A:SOP65P640X120-8N, symbol FS8205A:FS8205A
- removed R10: 100k MPPT Set Point, 0603 package, symbol Device:R
- removed R11: 0.05 Ohm Vishay Dale, 2512 package, symbol Device:R
- removed R12, R13, R16, R17: 100, symbol Device:R
- removed R7: 27.4k RFB1, 0603 package, symbol Device:R
- removed R8: 100k RFB2, 0603 package, symbol Device:R
- removed R9: 143k MPPT set point, 0603 package, symbol Device:R
- removed RT1: NCP18XH103F03RB, NCP18XH103F03RB:THRMC1608X95N, symbol NCP18XH103F03RB:NCP18XH103F03RB
- removed U2: LT3652EMSE_PBF, LT3652EMSE_PBF:MSOP-12_MSE, symbol LT3652EMSE_PBF:LT3652EMSE_PBF
- removed U3, U9: DW01A, DW01A:SOT95P280X145-6N, symbol DW01A:DW01A
- removed U6: ADS1015IRUGR, ADS1015IRUGR:IC_ADS1015IRUGR, symbol ADS1015IRUGR:ADS1015IRUGR
- removed U7: STPS140ZY, SOD123_2P8X1P7_STM, symbol 2026-09-20_06-34-23:STPS140ZY
- added U4: BQ29209DRBR, BQ29209DRBR:SON65P300X300X100-9N, symbol BQ29209DRBR:BQ29209DRBR
Connections:
- net GND: no longer BT4.2 (-)
- new net VSS: BT4.2 (-)
- no-connect marks 4 -> 2
Other:
- note removed: "Will need to have pull up resistors GPIO, SCL, SDA"

Commit message: Generate hierarchical schematic (8 sheets) from scripts/gen_schematic.py
- One sheet per block: solar_input, charger, battery, launch_inhibit,
  regulation, load_switches, telemetry, heater (DNP)
- Telemetry: INA228 + shunt in pack path, ADS1015 (ACS37612 dropped)
- Rails: 3.3 V / 5 V, LMZM33602 FB/RT/CFF from datasheet Table 7-1
- Fixes vs old flat schematic: TVS and boost diode were reversed
- ERC 0 violations; netlist matches expected_nets.json exactly
- Vendor pin-type fixes, deterministic footprint UUIDs, datasheet fetch script
- MISSING_PARTS.md, docs/CLAUDE.md/README updated for the decisions

Co-Authored-By: Claude Opus 5.5 <noreply@anthropic.com>
Parts:
- removed BT3: SM141K06L, SM141K06L:SOLAR_SM141K06L, symbol SM141K06L:SM141K06L
- removed BT4: Battery, symbol Device:Battery
- removed C5, C9: 10uF, symbol Device:C
- removed C6: C, symbol Device:C
- removed C8: GRM188R72A104KA35D, GRM188R72A104KA35D:CAPC1608X90N, symbol GRM188R72A104KA35D:GRM188R72A104KA35D
- removed CR2, CR3: CMSH3-40MA TR13 PBFREE, CR_SMA-CMSH3-40MA_CNS, symbol CSMH:CMSH3-40MA_TR13_PBFREE
- removed D3: SMBJ15A TVS DIODE 15VWM, symbol Device:D
- removed D4: SS34, SS34:DIOM7959X265N, symbol SS34:SS34
- removed L1: WE-PD_7332R, WE-PD_7332R:WE-PD_7332R, symbol WE-PD_7332R:WE-PD_7332R
- removed L3: 4.7µH, ≥3A, symbol Device:L
- removed R1, R21: 0.05 Ohm Vishay Dale, 2512 package, symbol Device:R
- removed R14, R5: 143k MPPT set point, 0603 package, symbol Device:R
- removed R15, R6: 100k MPPT Set Point, 0603 package, symbol Device:R
- removed R18, R4: 100k RFB2, 0603 package, symbol Device:R
- removed R19: 27.4k RFB1, 0603 package, symbol Device:R
- removed R2: 0ZCJ0100FF2E Bel Fuse, 0ZCJ0100FF2E:RESC3216X125N, symbol 0ZCJ0100FF2E:0ZCJ0100FF2E
- removed R3: 154k RFB1, 0603 package, symbol Device:R
- removed RT2: NCP18XH103F03RB, NCP18XH103F03RB:THRMC1608X95N, symbol NCP18XH103F03RB:NCP18XH103F03RB
- removed U1: LMZM33602RLRR, LMZM33602RLRR:VREG_LMZM33602RLRR, symbol LMZM33602RLRR:LMZM33602RLRR
- removed U10, U5: STPS140ZY, SOD123_2P8X1P7_STM, symbol 2026-09-20_06-34-23:STPS140ZY
- removed U4: BQ29209DRBR, BQ29209DRBR:SON65P300X300X100-9N, symbol BQ29209DRBR:BQ29209DRBR
- removed U8: LT3652EMSE_PBF, LT3652EMSE_PBF:MSOP-12_MSE, symbol LT3652EMSE_PBF:LT3652EMSE_PBF
Connections:
- no-connect marks 2 -> 0
Other:
- added sheet battery (sheets/battery.kicad_sch)
- added sheet charger (sheets/charger.kicad_sch)
- added sheet heater (sheets/heater.kicad_sch)
- added sheet launch_inhibit (sheets/launch_inhibit.kicad_sch)
- added sheet load_switches (sheets/load_switches.kicad_sch)
- added sheet regulation (sheets/regulation.kicad_sch)
- added sheet solar_input (sheets/solar_input.kicad_sch)
- added sheet telemetry (sheets/telemetry.kicad_sch)
- note added: "2S2P pack on Keystone clips + protection + current monitor"
- note added: "6xx load switches, 7xx telemetry, 8xx heater."
- note added: "Battery heater (optional, all DNP)"
- note added: "GND = P- (after the FS8205A cutoff FETs). BAT_N = cell negative, battery sheet only."
- note added: "LOBOSAT EPS - 2S2P Li-ion, solar charged. One sheet per block; inter-sheet nets are global labels."
- note added: "LT3652 solar MPPT charger (2S, 8.4 V float)"
- note added: "Launch inhibit / RBF"
- note added: "Open items: docs/06_open_questions.md and MISSING_PARTS.md. Values marked TBD are not decided."
- note added: "Power path: SOLAR_IN -> TVS + SS34 -> VSOLAR -> LT3652 -> VBUS <- PTC <- shunt <- fuse <- BAT_P (2S2P)"
- note added: "Rail A 3.3 V / Rail B 5 V (2x LMZM33602)"
- note added: "Reference designators: 1xx solar, 2xx charger, 3xx battery, 4xx inhibit, 5xx regulation,"
- note added: "Solar input + surge / backfeed protection"
- note added: "Subsystem load switches (3x TPS2553)"
- note added: "Telemetry: ADS1015 + MCU / OBC interface"
- note added: "VBUS -> launch inhibit (AO3401A) -> VBUS_SW -> LMZM33602 x2 -> RAIL_A 3.3 V / RAIL_B 5 V -> TPS2553 x3"
- note removed: "Boost cap"
- note removed: "Clamp Transients"
- note removed: "Decoupling Capacitor"
- note removed: "Solar Panels"
- note removed: "blocks reverse leakage back into the panel"
- note removed: "bootstraps the high-side driver"
- note removed: "catch diode"
- note removed: "thermistor for temperature, place near battery pack"
- company: (none) -> UNM Student Satellite Group - LOBOSAT
- title: (none) -> LOBOSAT EPS - top level

Commit message: Flatten schematic to a single A0 sheet
All 8 blocks on EPS_Lobosat_V1.kicad_sch, each in a titled dashed box;
local labels instead of global labels; sheets/ removed. Docs updated.
ERC 0 violations, netlist still matches expected_nets.json exactly.

Co-Authored-By: Claude Opus 5.5 <noreply@anthropic.com>
Parts:
- added BT301: 18650 cell 1A, Battery:BatteryHolder_Keystone_1042_1x18650, symbol Device:Battery_Cell
- added BT302: 18650 cell 1B, Battery:BatteryHolder_Keystone_1042_1x18650, symbol Device:Battery_Cell
- added BT303: 18650 cell 2A, Battery:BatteryHolder_Keystone_1042_1x18650, symbol Device:Battery_Cell
- added BT304: 18650 cell 2B, Battery:BatteryHolder_Keystone_1042_1x18650, symbol Device:Battery_Cell
- added C201: 10uF 50V X7R, Capacitor_SMD:C_1210_3225Metric, symbol Device:C
- added C202: TBD, Capacitor_SMD:C_0603_1608Metric, symbol Device:C
- added C203: 0.1uF 25V X7R, Capacitor_SMD:C_0603_1608Metric, symbol Device:C
- added C204: 10uF 25V X7R, Capacitor_SMD:C_1206_3216Metric, symbol Device:C
- added C301, C302, C303, C304, C305, C306, C601, C603, C605, C701, C702, C703, C704, C705, C801: 0.1uF, Capacitor_SMD:C_0603_1608Metric, symbol Device:C
- added C307: 0.33uF, Capacitor_SMD:C_0603_1608Metric, symbol Device:C
- added C501: 150pF, Capacitor_SMD:C_0603_1608Metric, symbol Device:C
- added C502, C503, C509, C510: 4.7uF 50V X7R, Capacitor_SMD:C_1210_3225Metric, symbol Device:C
- added C504, C505, C506, C507, C511, C512, C513, C514: 22uF 25V X7R, Capacitor_SMD:C_1210_3225Metric, symbol Device:C
- added C508: 100pF, Capacitor_SMD:C_0603_1608Metric, symbol Device:C
- added C602, C604, C606: 10uF 16V X7R, Capacitor_SMD:C_1206_3216Metric, symbol Device:C
- added D101: SMBJ15A, EPS_Footprints:DIOM4336X265N, symbol EPS_Symbols:SMBJ15A
- added D102: SS34, EPS_Footprints:DIOM7959X265N, symbol EPS_Symbols:SS34
- added D201: CMSH3-40MA, EPS_Footprints:CR_SMA-CMSH3-40MA_CNS, symbol EPS_Symbols:CMSH3-40MA
- added D202: STPS140ZY, EPS_Footprints:SOD123_2P8X1P7_STM, symbol EPS_Symbols:STPS140ZY
- added D801, D802: BAT54WS, Diode_SMD:D_SOD-323, symbol Device:D_Schottky
- added F301, F302, F303, F304, F305: TBD, Fuse:Fuse_1206_3216Metric, symbol Device:Fuse
- added F306: 0ZCJ0100FF2E, EPS_Footprints:RESC3216X125N, symbol EPS_Symbols:0ZCJ0100FF2E
- added J101: SOLAR_IN, Connector_JST:JST_PH_B2B-PH-K_1x02_P2.00mm_Vertical, symbol Connector_Generic:Conn_01x02
- added J601: OUT_VID, Connector_JST:JST_PH_B2B-PH-K_1x02_P2.00mm_Vertical, symbol Connector_Generic:Conn_01x02
- added J602: OUT_TLM, Connector_JST:JST_PH_B2B-PH-K_1x02_P2.00mm_Vertical, symbol Connector_Generic:Conn_01x02
- added J603: OUT_COM, Connector_JST:JST_PH_B2B-PH-K_1x02_P2.00mm_Vertical, symbol Connector_Generic:Conn_01x02
- added J701: MCU_IF, Connector_PinHeader_2.54mm:PinHeader_1x20_P2.54mm_Vertical, symbol Connector_Generic:Conn_01x20
- added L201: 4.7uH, EPS_Footprints:WE-PD_7332R, symbol EPS_Symbols:7447789004
- added Q201, Q202: TBD, Package_TO_SOT_SMD:SOT-23, symbol Transistor_FET:2N7002
- added Q301: FS8205A, EPS_Footprints:SOP65P640X120-8N, symbol EPS_Symbols:FS8205A
- added Q401: AO3401A, Package_TO_SOT_SMD:SOT-23, symbol Transistor_FET:AO3401A
- added Q801: AO3400A, Package_TO_SOT_SMD:SOT-23, symbol Transistor_FET:AO3400A
- added R201, R202, R203, R601, R603, R605, R808, R809, R810, R811: TBD, Resistor_SMD:R_0603_1608Metric, symbol Device:R
- added R204, R805: 1k, Resistor_SMD:R_0603_1608Metric, symbol Device:R
- added R205, R206, R401, R602, R604, R606, R803, R806: 100k, Resistor_SMD:R_0603_1608Metric, symbol Device:R
- added R207: 154k 1%, Resistor_SMD:R_0603_1608Metric, symbol Device:R
- added R208: 100k 1%, Resistor_SMD:R_0603_1608Metric, symbol Device:R
- added R209: 50m 1%, Resistor_SMD:R_2512_6332Metric, symbol Device:R
- added R301: 10m 1%, Resistor_SMD:R_2512_6332Metric, symbol Device:R
- added R302, R303: 470, Resistor_SMD:R_0603_1608Metric, symbol Device:R
- added R304: 2k, Resistor_SMD:R_0603_1608Metric, symbol Device:R
- added R305: 160, Resistor_SMD:R_0603_1608Metric, symbol Device:R
- added R306: 261 1%, Resistor_SMD:R_0603_1608Metric, symbol Device:R
- added R307, R308: 100, Resistor_SMD:R_0603_1608Metric, symbol Device:R
- added R309, R503, R506, R807: 10k 1%, Resistor_SMD:R_0603_1608Metric, symbol Device:R
- added R501: 133k 1%, Resistor_SMD:R_0603_1608Metric, symbol Device:R
- added R502: 23.2k 1%, Resistor_SMD:R_0603_1608Metric, symbol Device:R
- added R504: 88.7k 1%, Resistor_SMD:R_0603_1608Metric, symbol Device:R
- added R505: 40.2k 1%, Resistor_SMD:R_0603_1608Metric, symbol Device:R
- added R701: 330k 0.1%, Resistor_SMD:R_0603_1608Metric, symbol Device:R
- added R702: 47k 0.1%, Resistor_SMD:R_0603_1608Metric, symbol Device:R
- added R703: 200k 0.1%, Resistor_SMD:R_0603_1608Metric, symbol Device:R
- added R704, R705, R706: 100k 0.1%, Resistor_SMD:R_0603_1608Metric, symbol Device:R
- added R707, R708, R709, R710, R711, R712, R713, R714, R715, R804: 10k, Resistor_SMD:R_0603_1608Metric, symbol Device:R
- added R716, R717: 4.7k, Resistor_SMD:R_0603_1608Metric, symbol Device:R
- added R801, R802: TBD, Resistor_SMD:R_2512_6332Metric, symbol Device:R
- added SW401: SS-5GL, symbol Switch:SW_SPDT
- added TH201, TH301, TH801: 10k NTC, EPS_Footprints:THRMC1608X95N, symbol EPS_Symbols:NCP18XH103F03RB
- added U201: LT3652EMSE#PBF, EPS_Footprints:MSOP-12_MSE, symbol EPS_Symbols:LT3652EMSE_PBF
- added U301: INA228, EPS_Footprints:VSSOP10_DGS_TEX, symbol EPS_Symbols:INA228AIDGSR
- added U302: S-8252AAC-M6T1U, EPS_Footprints:SOT236-A-PKG_MP006-A-P-SD-2.1_ABL, symbol EPS_Symbols:S-8252AAC-M6T1U
- added U303: BQ29209DRBR, EPS_Footprints:SON65P300X300X100-9N, symbol EPS_Symbols:BQ29209DRBR
- added U501: LMZM33602 3V3, EPS_Footprints:VREG_LMZM33602RLRR, symbol EPS_Symbols:LMZM33602RLRR
- added U502: LMZM33602 5V, EPS_Footprints:VREG_LMZM33602RLRR, symbol EPS_Symbols:LMZM33602RLRR
- added U601, U602, U603: TPS2553DBVR, Package_TO_SOT_SMD:SOT-23-6, symbol EPS_Symbols:TPS2553DBVR
- added U701: ADS1015, EPS_Footprints:IC_ADS1015IRUGR, symbol EPS_Symbols:ADS1015IRUGR
- added U801: LM393, Package_SO:SOIC-8_3.9x4.9mm_P1.27mm, symbol Comparator:LM393
Connections:
- new net ADC_ALERT_N: J701.15 (Pin_15), R712.2, U701.2 (ALERT/RDY)
- new net ADC_BATMID: C704.1, R705.2, R706.1, U701.6 (AIN2)
- new net ADC_VBUS: C703.1, R703.2, R704.1, U701.5 (AIN1)
- new net ADC_VSOLAR: C702.1, R701.2, R702.1, U701.4 (AIN0)
- new net BAT_MID: BT303.2 (-), BT304.2 (-), F301.2, F302.2, R303.1, R306.1, R307.1, R705.1
- new net BAT_N: BT301.2 (-), BT302.2 (-), C302.2, C303.2, C305.2, C306.2, C307.2, Q301.2, Q301.3, U302.6 (VSS), U303.5 (GND), U303.6 (~{CB_EN}), U303.9 (EXP)
- new net BAT_P: F303.2, F304.2, F305.1, R302.1, R305.1, R308.1
- new net BAT_P_F: F305.2, R301.1, U301.10 (IN+)
- new net BAT_P_S: F306.1, R301.2, U301.9 (IN-)
- new net BQ_CD: C307.1, U303.4 (CD)
- new net BQ_VC1: C304.2, C305.1, R306.2, U303.2 (VC1)
- new net BQ_VC1CB: R307.2, U303.3 (VC1_CB)
- new net BQ_VC2: C304.1, R305.2, U303.1 (VC2)
- new net BQ_VDD: C306.1, R308.2, U303.7 (VDD)
- new net CELL1A_P: BT301.1 (+), F301.1
- new net CELL1B_P: BT302.1 (+), F302.1
- new net CELL2A_P: BT303.1 (+), F303.1
- new net CELL2B_P: BT304.1 (+), F304.1
- new net CHG_BOOST: C203.1, D202.1 (K), U201.11 (BOOST)
- new net CHG_FAULT_N: J701.13 (Pin_13), R711.2, U201.5 (*FAULT)
- new net CHG_G: Q301.5, U302.2 (CO)
- new net CHG_NTC: TH201.1, U201.8 (NTC)
- new net CHG_OVP: R204.1, U303.8 (OUT)
- new net CHG_OVP_G: Q201.1 (G), R204.2, R205.1
- new net CHG_SENSE: L201.2, R209.1, U201.10 (SENSE)
- new net CHG_SHDN: J701.14 (Pin_14), Q202.1 (G), R206.1
- new net CHG_SHDN_PIN: Q201.3 (D), Q202.3 (D), R203.2, U201.3 (*SHDN)
- new net CHG_STAT_N: J701.12 (Pin_12), R710.2, U201.4 (*CHRG)
- new net CHG_SW: C203.2, D201.1 (K), L201.1, U201.12 (SW)
- new net CHG_TIMER: C202.1, U201.6 (TIMER)
- new net CHG_VFB: R207.2, R208.1, U201.7 (VFB)
- new net CHG_VINREG: R201.2, R202.1, U201.2 (VIN_REG)
- new net DSG_G: Q301.4, U302.1 (DO)
- new net EN_COM: J701.8 (Pin_8), R606.1, U603.3 (EN)
- new net EN_TLM: J701.7 (Pin_7), R604.1, U602.3 (EN)
- new net EN_VID: J701.6 (Pin_6), R602.1, U601.3 (EN)
- new net FET_D: Q301.1, Q301.8
- new net FLT_COM_N: J701.11 (Pin_11), R709.2, U603.4 (~{FAULT})
- new net FLT_TLM_N: J701.10 (Pin_10), R708.2, U602.4 (~{FAULT})
- new net FLT_VID_N: J701.9 (Pin_9), R707.2, U601.4 (~{FAULT})
- new net GND: C201.2, C202.2, C204.2, C301.2, C502.2, C503.2, C504.2, C505.2, C506.2, C507.2, C509.2, C510.2, C511.2, C512.2, C513.2, C514.2, C601.2, C602.2, C603.2, C604.2, C605.2, C606.2, C701.2, C702.2, C703.2, C704.2, C705.2, C801.2, D101.2 (A), D201.2 (A), J101.2 (Pin_2), J601.2 (Pin_2), J602.2 (Pin_2), J603.2 (Pin_2), J701.2 (Pin_2), J701.20 (Pin_20), J701.5 (Pin_5), Q201.2 (S), Q202.2 (S), Q301.6, Q301.7, Q801.2 (S), R202.2, R205.2, R206.2, R208.2, R304.2, R601.2, R602.2, R603.2, R604.2, R605.2, R606.2, R702.2, R704.2, R706.2, R803.2, R806.2, R809.2, R811.2, SW401.2 (B), TH201.2, TH301.2, TH801.2, U201.13 (EPAD), U301.1 (A1), U301.2 (A0), U301.7 (GND), U501.14 (PGND__1), U501.15 (PGND__2), U501.18 (PGND__3), U501.5 (PGND), U501.PGND1 (PGND__4), U501.PGND10 (PGND__13), U501.PGND11 (PGND__14), U501.PGND12 (PGND__15), U501.PGND13 (PGND__16), U501.PGND14 (PGND__17), U501.PGND15 (PGND__18), U501.PGND16 (PGND__19), U501.PGND17 (PGND__20), U501.PGND18 (PGND__21), U501.PGND19 (PGND__22), U501.PGND2 (PGND__5), U501.PGND20 (PGND__23), U501.PGND21 (PGND__24), U501.PGND22 (PGND__25), U501.PGND23 (PGND__26), U501.PGND24 (PGND__27), U501.PGND25 (PGND__28), U501.PGND26 (PGND__29), U501.PGND27 (PGND__30), U501.PGND28 (PGND__31), U501.PGND29 (PGND__32), U501.PGND3 (PGND__6), U501.PGND30 (PGND__33), U501.PGND31 (PGND__34), U501.PGND32 (PGND__35), U501.PGND4 (PGND__7), U501.PGND5 (PGND__8), U501.PGND6 (PGND__9), U501.PGND7 (PGND__10), U501.PGND8 (PGND__11), U501.PGND9 (PGND__12), U502.14 (PGND__1), U502.15 (PGND__2), U502.18 (PGND__3), U502.5 (PGND), U502.PGND1 (PGND__4), U502.PGND10 (PGND__13), U502.PGND11 (PGND__14), U502.PGND12 (PGND__15), U502.PGND13 (PGND__16), U502.PGND14 (PGND__17), U502.PGND15 (PGND__18), U502.PGND16 (PGND__19), U502.PGND17 (PGND__20), U502.PGND18 (PGND__21), U502.PGND19 (PGND__22), U502.PGND2 (PGND__5), U502.PGND20 (PGND__23), U502.PGND21 (PGND__24), U502.PGND22 (PGND__25), U502.PGND23 (PGND__26), U502.PGND24 (PGND__27), U502.PGND25 (PGND__28), U502.PGND26 (PGND__29), U502.PGND27 (PGND__30), U502.PGND28 (PGND__31), U502.PGND29 (PGND__32), U502.PGND3 (PGND__6), U502.PGND30 (PGND__33), U502.PGND31 (PGND__34), U502.PGND32 (PGND__35), U502.PGND4 (PGND__7), U502.PGND5 (PGND__8), U502.PGND6 (PGND__9), U502.PGND7 (PGND__10), U502.PGND8 (PGND__11), U502.PGND9 (PGND__12), U601.2 (GND), U602.2 (GND), U603.2 (GND), U701.1 (ADDR), U701.3 (GND), U801.4 (V-)
- new net HEATER_EN: J701.17 (Pin_17), R805.1, R806.1
- new net HTR_COLD: D801.2 (A), R804.2, U801.1
- new net HTR_EN_R: D802.2 (A), R805.2
- new net HTR_GATE: D801.1 (K), D802.1 (K), Q801.1 (G), R803.1, U801.7
- new net HTR_NTC: R807.2, TH801.1, U801.3 (+), U801.5 (+)
- new net HTR_SW: Q801.3 (D), R801.2, R802.2
- new net HTR_VCOLD: R808.2, R809.1, U801.2 (-)
- new net HTR_VHOT: R810.2, R811.1, U801.6 (-)
- new net I2C_SCL: J701.4 (Pin_4), R717.2, U301.5 (SCL), U701.10 (SCL)
- new net I2C_SDA: J701.3 (Pin_3), R716.2, U301.4 (SDA), U701.9 (SDA)
- new net INA_ALERT_N: J701.16 (Pin_16), R713.2, U301.3 (ALERT)
- new net INH_GATE: Q401.1 (G), R401.1, SW401.1 (A)
- new net LSW_COM_ILIM: R605.1, U603.5 (ILIM)
- new net LSW_TLM_ILIM: R603.1, U602.5 (ILIM)
- new net LSW_VID_ILIM: R601.1, U601.5 (ILIM)
- new net NTC_BAT: C705.1, R309.2, TH301.1, U701.7 (AIN3)
- new net PG_RAIL_A: J701.18 (Pin_18), R714.2, U501.17 (PGOOD)
- new net PG_RAIL_B: J701.19 (Pin_19), R715.2, U502.17 (PGOOD)
- new net PWR_COM: C606.1, J603.1 (Pin_1), U603.6 (OUT)
- new net PWR_TLM: C604.1, J602.1 (Pin_1), U602.6 (OUT)
- new net PWR_VID: C602.1, J601.1 (Pin_1), U601.6 (OUT)
- new net RAIL_A: C301.1, C501.1, C504.1, C505.1, C506.1, C507.1, C601.1, C603.1, C701.1, J701.1 (Pin_1), R309.1, R502.1, R707.1, R708.1, R709.1, R710.1, R711.1, R712.1, R713.1, R714.1, R715.1, R716.1, R717.1, R804.1, R807.1, R808.1, R810.1, U301.6 (VS), U501.6 (VOUT), U501.7 (VOUT__1), U501.8 (VOUT__2), U501.VOUT1 (VOUT__3), U501.VOUT10 (VOUT__12), U501.VOUT11 (VOUT__13), U501.VOUT12 (VOUT__14), U501.VOUT13 (VOUT__15), U501.VOUT14 (VOUT__16), U501.VOUT15 (VOUT__17), U501.VOUT16 (VOUT__18), U501.VOUT17 (VOUT__19), U501.VOUT18 (VOUT__20), U501.VOUT19 (VOUT__21), U501.VOUT2 (VOUT__4), U501.VOUT3 (VOUT__5), U501.VOUT4 (VOUT__6), U501.VOUT5 (VOUT__7), U501.VOUT6 (VOUT__8), U501.VOUT7 (VOUT__9), U501.VOUT8 (VOUT__10), U501.VOUT9 (VOUT__11), U601.1 (IN), U602.1 (IN), U701.8 (VDD)
- new net RAIL_B: C508.1, C511.1, C512.1, C513.1, C514.1, C605.1, R505.1, U502.6 (VOUT), U502.7 (VOUT__1), U502.8 (VOUT__2), U502.VOUT1 (VOUT__3), U502.VOUT10 (VOUT__12), U502.VOUT11 (VOUT__13), U502.VOUT12 (VOUT__14), U502.VOUT13 (VOUT__15), U502.VOUT14 (VOUT__16), U502.VOUT15 (VOUT__17), U502.VOUT16 (VOUT__18), U502.VOUT17 (VOUT__19), U502.VOUT18 (VOUT__20), U502.VOUT19 (VOUT__21), U502.VOUT2 (VOUT__4), U502.VOUT3 (VOUT__5), U502.VOUT4 (VOUT__6), U502.VOUT5 (VOUT__7), U502.VOUT6 (VOUT__8), U502.VOUT7 (VOUT__9), U502.VOUT8 (VOUT__10), U502.VOUT9 (VOUT__11), U603.1 (IN)
- new net REGA_AGND: R501.2, R503.2, U501.1 (AGND)
- new net REGA_FB: C501.2, R502.2, R503.1, U501.16 (FB)
- new net REGA_RT: R501.1, U501.3 (RT)
- new net REGA_SW: U501.10 (SW__1), U501.11 (SW__2), U501.9 (SW)
- new net REGB_AGND: R504.2, R506.2, U502.1 (AGND)
- new net REGB_FB: C508.2, R505.2, R506.1, U502.16 (FB)
- new net REGB_RT: R504.1, U502.3 (RT)
- new net REGB_SW: U502.10 (SW__1), U502.11 (SW__2), U502.9 (SW)
- new net S8252_VC: C303.1, R303.2, U302.4 (VC)
- new net S8252_VDD: C302.1, R302.2, U302.5 (VDD)
- new net S8252_VM: R304.1, U302.3 (VM)
- new net VBUS: C204.1, C801.1, D202.2 (A), F306.2, Q401.2 (S), R207.1, R209.2, R401.2, R703.1, R801.1, R802.1, U201.9 (BAT), U301.8 (VBUS), U801.8 (V+)
- new net VBUS_SW: C502.1, C503.1, C509.1, C510.1, Q401.3 (D), U501.2 (EN/SYNC), U501.4 (VIN), U502.2 (EN/SYNC), U502.4 (VIN)
- new net VSOLAR: C201.1, D102.C, R201.1, R203.1, R701.1, U201.1 (VIN)
- new net VSOLAR_RAW: D101.1 (K), D102.A, J101.1 (Pin_1)
- no-connect marks 0 -> 1
Other:
- removed sheet battery
- removed sheet charger
- removed sheet heater
- removed sheet launch_inhibit
- removed sheet load_switches
- removed sheet regulation
- removed sheet solar_input
- removed sheet telemetry
- note added: "1 RAIL_A 2 GND 3 SDA 4 SCL 5 GND 6 EN_VID 7 EN_TLM 8 EN_COM 9 FLT_VID_N 10 FLT_TLM_N"
- note added: "11 FLT_COM_N 12 CHG_STAT_N 13 CHG_FAULT_N 14 CHG_SHDN 15 ADC_ALERT_N 16 INA_ALERT_N"
- note added: "17 HEATER_EN 18 PG_RAIL_A 19 PG_RAIL_B 20 GND"
- note added: "2S2P PACK ON KEYSTONE CLIPS + PROTECTION + CURRENT MONITOR"
- note added: "7xx telemetry, 8xx heater. Open items: docs/06_open_questions.md and MISSING_PARTS.md. TBD = not decided."
- note added: "ADS1015 at 0x48 (ADDR = GND), VDD = RAIL_A 3.3 V. Use FSR +/-4.096 V; inputs must stay <= VDD."
- note added: "AGND must NOT be tied to PGND externally (datasheet 5): each module has its own AGND net."
- note added: "AIN0 VSOLAR x 47/377 (15 V -> 1.87 V, TVS clamp 24 V -> 3.0 V) AIN1 VBUS x 1/3 (8.4 V -> 2.8 V)"
- note added: "AIN2 BAT_MID x 1/2 (4.2 V -> 2.1 V) AIN3 NTC_BAT. Battery current/voltage come from the INA228."
- note added: "AO3401A Vgs max +/-12 V; pack max 8.4 V so no gate zener fitted."
- note added: "All parts DNP until the heater decision (docs/06 #6). Thresholds TBD."
- note added: "BATTERY HEATER (OPTIONAL, ALL DNP)"
- note added: "Charge current = 100 mV / R_SENSE = 2 A with 50 mOhm (verify against LT3652 datasheet)."
- note added: "D801/D802 (BAT54WS) were added to make the OR; not in the kit parts list."
- note added: "EN tied to VIN (allowed by datasheet). Add an EN divider later if you want a UVLO."
- note added: "FIXED vs old schematic: STPS140ZY boost diode was reversed; anode must be on BAT (VBUS)."
- note added: "FIXED vs old schematic: TVS was reversed (cathode on GND) and would have shorted the panel."
- note added: "Fuse/PTC ratings TBD (docs/06 #4). Shunt 10 mOhm: 4 A -> 40 mV = INA228 ADCRANGE=1 full scale."
- note added: "GND = P- (after the FS8205A cutoff FETs). BAT_N = cell negative (battery block only)."
- note added: "Gate pulled up to VBUS = FET off by default. Switch NC contact closes INH_GATE -> GND when the"
- note added: "Ground reference: S-8252 and BQ29209 sit on BAT_N (cell negative). Everything else is on GND (P-)."
- note added: "Heater ON = (too cold OR HEATER_EN) AND NOT too hot."
- note added: "ILIM resistors TBD (docs/06 #5): 15k..232k, see TPS2553 datasheet Fig. 23."
- note added: "INA228 address 0x40 (A0 = A1 = GND). ACS37612 dropped (decision 2026-10-23)."
- note added: "Keystone 1042 holder footprint from KiCad library; exact clip MPN TBD (docs/06 #10)."
- note added: "LAUNCH INHIBIT / RBF"
- note added: "LM393 runs from VBUS: its input common-mode range is only up to Vcc - 1.5 V."
- note added: "LOBOSAT EPS - 2S2P Li-ion, solar charged. Single sheet; each box is one block. Same label text = same net."
- note added: "LT3652 SOLAR MPPT CHARGER (2S, 8.4 V FLOAT)"
- note added: "MCU connector pin order (placeholder 1x20 header, real connector TBD docs/06 #8):"
- note added: "N-FET that pulls SHDN low. Inverter FET part TBD (#9)."
- note added: "No hysteresis yet: add a feedback resistor per comparator when thresholds are chosen."
- note added: "Note: the BAT_MID divider draws ~21 uA from the bottom cells only; BQ29209 balancing covers it."
- note added: "Only ONE inhibit built; count depends on the launch provider (docs/06 #7)."
- note added: "Only the FS8205A joins BAT_N and GND. FET1 (G1) = discharge, FET2 (G2) = charge."
- note added: "Open: string Voc must stay below 15 V for SMBJ15A (docs/06 #2). Connector type TBD (#8)."
- note added: "Output caps 10 uF chosen (datasheet: 0.1 uF min on IN; output cap per load)."
- note added: "Panel string -> TVS clamp -> SS34 blocking diode -> VSOLAR (charger input)."
- note added: "Per-cell fuses F301-F304 are FITTED, not DNP: DNP would open each cell. Use 0 Ohm 1206 if unwanted."
- note added: "Pins 12/13 are DNC (no symbol pin). SW pins only go to a small copper island."
- note added: "RAIL A 3.3 V / RAIL B 5 V (2X LMZM33602)"
- note added: "RT 133k (300 kHz), COUT >= 88 uF; 5 V -> RFBT 40.2k, CFF 100 pF, RT 88.7k (450 kHz), COUT >= 66 uF."
- note added: "Rail assignment default: VID, TLM on RAIL_A (3.3 V); COM on RAIL_B (5 V). Output connectors TBD (#8)."
- note added: "Reference designators: 1xx solar, 2xx charger, 3xx battery, 4xx inhibit, 5xx regulation, 6xx load switches,"
- note added: "SHDN: BQ29209 OUT (CHG_OVP, high = overvoltage) and MCU CHG_SHDN (high = stop) each drive an"
- note added: "SOLAR INPUT + SURGE / BACKFEED PROTECTION"
- note added: "SS-5GL has SOLDER terminals; for PCB mounting consider SS-5GLD. No footprint yet (MISSING_PARTS)."
- note added: "SS34 footprint is SMC (DIOM7959) from SnapEDA; parts list said SMA. Pick one before ordering."
- note added: "SUBSYSTEM LOAD SWITCHES (3X TPS2553)"
- note added: "Symbol pin map: 2 = COM, 1 = NC, 3 = NO (verify against the switch you buy)."
- note added: "TBD: VIN_REG divider (docs/06 #3, old 143k/100k was for 1S), TIMER cap, SHDN pull-up (#9)."
- note added: "TELEMETRY: ADS1015 + MCU / OBC INTERFACE"
- note added: "TPS2553 (not -1): EN active HIGH, auto-retry. 100k EN pull-downs keep loads off until the MCU says so."
- note added: "U801A: NTC node above V_COLD -> output released -> D801 pulls the gate up."
- note added: "U801B: NTC node below V_HOT -> output low -> forces the gate low (overrides both)."
- note added: "VFB divider 154k/100k: 3.3 V x (1 + 154/100) = 8.38 V float. Verify the datasheet's bias-current"
- note added: "Values from LMZM33602 datasheet Table 7-1 (RFBB = 10k): 3.3 V -> RFBT 23.2k, CFF 150 pF,"
- note added: "WARNING: datasheet recommends VIN >= 1.3 x VOUT = 6.5 V for the 5 V rail; pack goes to 6.0 V."
- note added: "correction (LT3652 datasheet could not be downloaded automatically - put 3652fe.pdf in datasheets/)."
- note added: "lever is released (deployed) = FET on. Stowed / RBF inserted = lever pressed = NC open = off."
- note removed: "2S2P pack on Keystone clips + protection + current monitor"
- note removed: "6xx load switches, 7xx telemetry, 8xx heater."
- note removed: "Battery heater (optional, all DNP)"
- note removed: "GND = P- (after the FS8205A cutoff FETs). BAT_N = cell negative, battery sheet only."
- note removed: "LOBOSAT EPS - 2S2P Li-ion, solar charged. One sheet per block; inter-sheet nets are global labels."
- note removed: "LT3652 solar MPPT charger (2S, 8.4 V float)"
- note removed: "Launch inhibit / RBF"
- note removed: "Open items: docs/06_open_questions.md and MISSING_PARTS.md. Values marked TBD are not decided."
- note removed: "Rail A 3.3 V / Rail B 5 V (2x LMZM33602)"
- note removed: "Reference designators: 1xx solar, 2xx charger, 3xx battery, 4xx inhibit, 5xx regulation,"
- note removed: "Solar input + surge / backfeed protection"
- note removed: "Subsystem load switches (3x TPS2553)"
- note removed: "Telemetry: ADS1015 + MCU / OBC interface"
- title: LOBOSAT EPS - top level -> LOBOSAT EPS

Commit message: Hand-tidied single-sheet schematic, drop heater, add BOM and README
- Schematic tidied by hand in KiCad (one A0 sheet); rail B regulator block
  rebuilt (now U503 + R507-R509, C515-C521), heater block removed
- Fixed copy-paste labels on U503: SW pins were on REGA_SW (shorted both
  regulators' switch nodes) and PGOOD on PG_RAIL_A
- ERC 0 violations; expected_nets.json reset to the verified netlist
- BOM.csv exported from the schematic (62 lines, 121 parts)
- README: what changed, why values are TBD, full BOM table
- Generator retired to scripts/archive/ (would overwrite manual edits)

Co-Authored-By: Claude Opus 5.5 <noreply@anthropic.com>
Parts:
- removed C508: 100pF, Capacitor_SMD:C_0603_1608Metric, symbol Device:C
- removed C509, C510: 4.7uF 50V X7R, Capacitor_SMD:C_1210_3225Metric, symbol Device:C
- removed C511, C512, C513, C514: 22uF 25V X7R, Capacitor_SMD:C_1210_3225Metric, symbol Device:C
- removed C801: 0.1uF, Capacitor_SMD:C_0603_1608Metric, symbol Device:C
- removed D801, D802: BAT54WS, Diode_SMD:D_SOD-323, symbol Device:D_Schottky
- removed Q801: AO3400A, Package_TO_SOT_SMD:SOT-23, symbol Transistor_FET:AO3400A
- removed R504: 88.7k 1%, Resistor_SMD:R_0603_1608Metric, symbol Device:R
- removed R505: 40.2k 1%, Resistor_SMD:R_0603_1608Metric, symbol Device:R
- removed R506, R807: 10k 1%, Resistor_SMD:R_0603_1608Metric, symbol Device:R
- removed R801, R802: TBD, Resistor_SMD:R_2512_6332Metric, symbol Device:R
- removed R803, R806: 100k, Resistor_SMD:R_0603_1608Metric, symbol Device:R
- removed R804: 10k, Resistor_SMD:R_0603_1608Metric, symbol Device:R
- removed R805: 1k, Resistor_SMD:R_0603_1608Metric, symbol Device:R
- removed R808, R809, R810, R811: TBD, Resistor_SMD:R_0603_1608Metric, symbol Device:R
- removed TH801: 10k NTC, EPS_Footprints:THRMC1608X95N, symbol EPS_Symbols:NCP18XH103F03RB
- removed U502: LMZM33602 5V, EPS_Footprints:VREG_LMZM33602RLRR, symbol EPS_Symbols:LMZM33602RLRR
- removed U801: LM393, Package_SO:SOIC-8_3.9x4.9mm_P1.27mm, symbol Comparator:LM393
- added C515, C516: 4.7uF 50V X7R, Capacitor_SMD:C_1210_3225Metric, symbol Device:C
- added C517: 100pF, Capacitor_SMD:C_0603_1608Metric, symbol Device:C
- added C518, C519, C520, C521: 22uF 25V X7R, Capacitor_SMD:C_1210_3225Metric, symbol Device:C
- added R507: 40.2k 1%, Resistor_SMD:R_0603_1608Metric, symbol Device:R
- added R508: 88.7k 1%, Resistor_SMD:R_0603_1608Metric, symbol Device:R
- added R509: 10k 1%, Resistor_SMD:R_0603_1608Metric, symbol Device:R
- added U503: LMZM33602 3V3, EPS_Footprints:VREG_LMZM33602RLRR, symbol EPS_Symbols:LMZM33602RLRR
Connections:
- net CELL2A_P: now also F304.1; no longer F303.1
- net CELL2B_P: now also F303.1; no longer F304.1
- net CHG_SENSE: now also L201.1; no longer L201.2
- net CHG_SW: now also L201.2; no longer L201.1
- net CHG_VINREG: now also R201.1; no longer R201.2
- net GND: now also C515.2, C516.2, C518.2, C519.2, C520.2, C521.2, U503.14 (PGND__1), U503.15 (PGND__2), U503.18 (PGND__3), U503.5 (PGND), U503.PGND1 (PGND__4), U503.PGND10 (PGND__13), U503.PGND11 (PGND__14), U503.PGND12 (PGND__15), U503.PGND13 (PGND__16), U503.PGND14 (PGND__17), U503.PGND15 (PGND__18), U503.PGND16 (PGND__19), U503.PGND17 (PGND__20), U503.PGND18 (PGND__21), U503.PGND19 (PGND__22), U503.PGND2 (PGND__5), U503.PGND20 (PGND__23), U503.PGND21 (PGND__24), U503.PGND22 (PGND__25), U503.PGND23 (PGND__26), U503.PGND24 (PGND__27), U503.PGND25 (PGND__28), U503.PGND26 (PGND__29), U503.PGND27 (PGND__30), U503.PGND28 (PGND__31), U503.PGND29 (PGND__32), U503.PGND3 (PGND__6), U503.PGND30 (PGND__33), U503.PGND31 (PGND__34), U503.PGND32 (PGND__35), U503.PGND4 (PGND__7), U503.PGND5 (PGND__8), U503.PGND6 (PGND__9), U503.PGND7 (PGND__10), U503.PGND8 (PGND__11), U503.PGND9 (PGND__12)
- net PG_RAIL_B: now also U503.17 (PGOOD)
- net RAIL_B: now also C517.1, C518.1, C519.1, C520.1, C521.1, R507.1, U503.6 (VOUT), U503.7 (VOUT__1), U503.8 (VOUT__2), U503.VOUT1 (VOUT__3), U503.VOUT10 (VOUT__12), U503.VOUT11 (VOUT__13), U503.VOUT12 (VOUT__14), U503.VOUT13 (VOUT__15), U503.VOUT14 (VOUT__16), U503.VOUT15 (VOUT__17), U503.VOUT16 (VOUT__18), U503.VOUT17 (VOUT__19), U503.VOUT18 (VOUT__20), U503.VOUT19 (VOUT__21), U503.VOUT2 (VOUT__4), U503.VOUT3 (VOUT__5), U503.VOUT4 (VOUT__6), U503.VOUT5 (VOUT__7), U503.VOUT6 (VOUT__8), U503.VOUT7 (VOUT__9), U503.VOUT8 (VOUT__10), U503.VOUT9 (VOUT__11)
- net REGA_AGND: now also R501.1, R503.1; no longer R501.2, R503.2
- net REGA_FB: now also R503.2; no longer R503.1
- net REGA_RT: now also R501.2; no longer R501.1
- net REGB_AGND: now also R508.1, R509.1, U503.1 (AGND)
- net REGB_FB: now also C517.2, R507.2, R509.2, U503.16 (FB)
- net REGB_RT: now also R508.2, U503.3 (RT)
- net REGB_SW: now also U503.10 (SW__1), U503.11 (SW__2), U503.9 (SW)
- net VBUS_SW: now also C515.1, C516.1, U503.2 (EN/SYNC), U503.4 (VIN)
- net VSOLAR: now also R201.2; no longer R201.1
- net HEATER_EN: no longer names the net of J701.17 (Pin_17)
- no-connect marks 1 -> 2
Other:
- note removed: "All parts DNP until the heater decision (docs/06 #6). Thresholds TBD."
- note removed: "BATTERY HEATER (OPTIONAL, ALL DNP)"
- note removed: "D801/D802 (BAT54WS) were added to make the OR; not in the kit parts list."
- note removed: "Heater ON = (too cold OR HEATER_EN) AND NOT too hot."
- note removed: "LM393 runs from VBUS: its input common-mode range is only up to Vcc - 1.5 V."
- note removed: "No hysteresis yet: add a feedback resistor per comparator when thresholds are chosen."
- note removed: "U801A: NTC node above V_COLD -> output released -> D801 pulls the gate up."
- note removed: "U801B: NTC node below V_HOT -> output low -> forces the gate low (overrides both)."
- moved on the sheet: BT301, BT302, BT303, BT304, C201, C202, C203, C204, C301, C302, C303, C304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

Commit message: Switch small resistors and capacitors from 0603 to 0805
65 parts (46 R, 19 C) for easier hand soldering. 1206/1210 bulk caps,
2512 shunts, 1206 fuses and 0603 NCP18 thermistors unchanged.
ERC 0 violations, netlist unchanged (check_netlist PASS), BOM re-exported.

Co-Authored-By: Claude Opus 5.5 <noreply@anthropic.com>
Parts:
- C202, C203, C301, C302, C303, C304, C305, C306, C307, C501, C517, C601, C603, C605, C701, C702, C703, C704, C705: footprint Capacitor_SMD:C_0603_1608Metric -> Capacitor_SMD:C_0805_2012Metric
- R201, R202, R203, R204, R205, R206, R207, R208, R302, R303, R304, R305, R306, R307, R308, R309, R401, R501, R502, R503, R507, R508, R509, R601, R602, R603, R604, R605, R606, R701, R702, R703, R704, R705, R706, R707, R708, R709, R710, R711, R712, R713, R714, R715, R716, R717: footprint Resistor_SMD:R_0603_1608Metric -> Resistor_SMD:R_0805_2012Metric
